File: hardware/kicad/modules/default/module.kicad_sch (KiCad schematic)
At the start: 42 parts, among them J1 MOD_CONN, J10 MOD_CONN, J11 MOD_CONN, J12 MOD_CONN, J13 MOD_CONN, J14 MOD_CONN, J15 MOD_CONN, J16 MOD_CONN, J17 MOD_CONN, J18 MOD_CONN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

Commit message: improve module silkscreen
Changed lines of the file:
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@@
 (kicad_sch
-	(version 20231120)
+	(version 20250114)
 	(generator "eeschema")
-	(generator_version "8.0")
+	(generator_version "9.0")
 	(paper "A4")
+	(text "RGB Led\n"
+		(exclude_from_sim no)
+		(at 108.966 48.768 0)
+		(effects
+			(font
+				(size 1.778 1.778)
+			)
+		)
+	)
+	(text "Button\n"
+		(exclude_from_sim no)
+		(at 41.656 126.238 0)
+		(effects
+			(font
+				(size 1.778 1.778)
+			)
+		)
+	)
+	(text "Module"
+		(exclude_from_sim no)
+		(at 40.132 94.488 0)
+		(effects
+			(font
+				(size 1.778 1.778)
+			)
+		)
+	)
 	(polyline
 		(pts
@@
 		)
 	)
-	(text "RGB Led\n"
-		(exclude_from_sim no)
-		(at 108.966 48.768 0)
-		(effects
-			(font
-				(size 1.778 1.778)
-			)
-		)
-	)
-	(text "Button\n"
-		(exclude_from_sim no)
-		(at 41.656 126.238 0)
-		(effects
-			(font
-				(size 1.778 1.778)
-			)
-		)
-	)
-	(text "Module"
-		(exclude_from_sim no)
-		(at 40.132 94.488 0)
-		(effects
-			(font
-				(size 1.778 1.778)
-			)
-		)
-	)
 	(global_label "MOSI"
 		(shape input)
@@
 		)
 	)
+	(embedded_fonts no)
 )
